File: ESP32_charger/ESP32_charger.kicad_sch (KiCad schematic)
At the start: 60 parts, among them J1 USB_C_Receptacle_USB2.0_16P, J2 Conn_01x04_Pin, Q2 BC817W, Q3 HL-2301V, SW1 SW_Push, SW2 SW_Push, U1 ESP32-WROOM-32, U2 XM5062S, U3 HT2348ARTZ8, U4 INA219AxDCN

Commit message: update to order version
placed silkscreen
placed logos
add 3d models
generate 3d model
Parts:
- SW1, SW2: footprint TheBrutzlers_Lib:microswitch -> Button_Switch_SMD:SW_SPST_CK_RS282G05A3
Changed lines of the file:
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@@
 		(dnp no)
 		(property "Reference" "FB1"
-			(at 41.275 21.59 90)
+			(at 41.91 17.78 90)
 			(effects
 				(font
@@
 			)
 		)
-		(property "Footprint" "TheBrutzlers_Lib:microswitch"
+		(property "Footprint" "Button_Switch_SMD:SW_SPST_CK_RS282G05A3"
 			(at 106.68 91.44 0)
 			(effects
@@
 		(dnp no)
 		(property "Reference" "D1"
-			(at 48.895 21.59 0)
+			(at 50.8 16.51 0)
 			(effects
 				(font
@@
 		)
 		(property "Value" "D"
-			(at 47.625 17.78 0)
+			(at 53.34 17.78 0)
 			(effects
 				(font
@@
 			)
 		)
-		(property "Footprint" "TheBrutzlers_Lib:microswitch"
+		(property "Footprint" "Button_Switch_SMD:SW_SPST_CK_RS282G05A3"
 			(at 106.68 96.52 0)
 			(effects
